File: CM108B/CM108B.kicad_sch (KiCad schematic)
At the start: 4 parts, among them J1 USB_A, SW1 MST22D18G2, SW2 MST22D18G2, U1 CM108B

Commit message: Completed more connections WIP
Parts:
- added C1, C2: 100uF, symbol Device:C_Polarized
- added C3: 1uF, symbol Device:C
- added C4: 100nF, symbol Device:C
- added C5, C6: 100pF, symbol Device:C
- added R1, R2: 39R, symbol Device:R
- added SW3, SW4, SW5, SW6: C4B1802110, easyeda2kicad:SW-SMD_4P-L3.5-W3.0-P1.50-LS4.7, symbol Push Switch:C4B1802110
Connections:
- net GND: now also U1.24 (AVSS), U1.36 (DVSS), C3.2, C4.2, SW3.3, SW3.4, SW4.3, SW4.4, SW5.3, SW5.4, SW6.3, SW6.4
- net MODE: now reaches SW1.2, SW1.5, U1.10 (MODE)
- net MUTEP: now reaches U1.18 (MUTEP)
- net MUTEP: now also SW6.1, SW6.2
- net LOL: now reaches U1.30 (LOL)
- net LOL: now also C2.1
- net LOBS: now reaches U1.31 (LOBS)
- net LOR: now reaches U1.32 (LOR)
- net LOR: now also C1.1
- net MSEL: now reaches SW2.2, SW2.5, U1.38 (MSEL)
- net VOLUP: now reaches U1.39 (VOLUP)
- net VOLUP: now also SW5.1, SW5.2
- net VOLDN: now reaches U1.48 (VOLDN)
- net VOLDN: now also SW4.1, SW4.2
- net MUTER: now reaches U1.6 (MUTER)
- net MUTER: now also SW3.1, SW3.2
- net DREG18: now reaches U1.8 (DREG18)
- net DREG18: now also C3.1
- net DREG33: now reaches U1.9 (DREG33)
- net DREG33: now also C4.1
- new net: C6.1, R2.2
- new net: C2.2, R2.1
- new net: C1.2, R1.1
- new net: C5.1, R1.2
- no-connect marks 2 -> 18
Other:
- moved on the sheet: J1, SW1
