File: MX26631DL/MX26631DL.kicad_pcb (KiCad board)
At the start: 2 copper layers, 21 x 21 mm, 15 parts, among them U1 ZX-PZ2.54-1-1PZZ, U2 ZX-PZ2.54-1-1PZZ, U3 TPESD0402G15V, U4 MX26631DL

Commit message: New iteration done
Parts:
- moved U1 5.83 mm to (97.9, 82.3)
- moved U2 4.89 mm to (97.9, 104.1)
Routing:
- net /+5V_unprot: track 20.7 -> 26.2 mm
Other:
- board size 21 x 21 mm -> 21 x 31 mm
Changed lines of the file:
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@@
 	(footprint "easyeda2kicad:HDR-TH_1P-P2.54-V-M"
 		(layer "F.Cu")
-		(at 97.9 88.1)
+		(at 97.87 82.27)
 		(property "Reference" "U1"
 			(at 0 -2.248 0)
@@
 	(footprint "easyeda2kicad:HDR-TH_1P-P2.54-V-M"
 		(layer "F.Cu")
-		(at 97.9 99.175)
+		(at 97.9 104.07)
 		(property "Reference" "U2"
 			(at 0.144 -2.147 0)
@@
 	)
 	(gr_rect
-		(start 95 83)
-		(end 116 104)
+		(start 95 78)
+		(end 116 109)
 		(stroke
 			(width 0.05)
@@
 		(layer "User.1")
 		(pts
-			(xy 116 102.5) (xy 95 102.5)
+			(xy 116 109) (xy 95 109)
 		)
-		(height 5.375)
+		(height 2.77)
 		(orientation 0)
 		(format
@@
 		)
 		(gr_text "21"
-			(at 105.5 106.725 0)
+			(at 105.5 110.62 0)
 			(layer "User.1")
 			(effects
@@
 		(layer "User.1")
 		(pts
-			(xy 116 83) (xy 116 104)
+			(xy 116 78) (xy 116 109)
 		)
 		(height 3.4)
@@
 			(keep_text_aligned yes)
 		)
-		(gr_text "21"
+		(gr_text "31"
 			(at 118.25 93.5 90)
 			(layer "User.1")
@@
 	)
 	(segment
-		(start 101.473 92.964)
-		(end 102.459 92.964)
+		(start 97.87 82.27)
+		(end 97.87 88.67)
 		(width 0.4)
 		(layer "F.Cu")
@@
 	)
 	(segment
-		(start 97.9 88.1)
-		(end 97.9 89.391)
-		(width 0.4)
-		(layer "F.Cu")
-		(net 1)
-	)
-	(segment
-		(start 97.9 89.391)
-		(end 101.473 92.964)
+		(start 102.164 92.964)
+		(end 102.459 92.964)
 		(width 0.4)
 		(layer "F.Cu")
@@
 	)
 	(segment
+		(start 97.87 88.67)
+		(end 102.164 92.964)
+		(width 0.4)
+		(layer "F.Cu")
+		(net 1)
+	)
+	(segment
 		(start 111.5 98.175)
 		(end 112.6 98.175)
@@
 		(polygon
 			(pts
-				(xy 94.975 82.975) (xy 116 82.975) (xy 116 104.025) (xy 94.975 104.025)
+				(xy 94.975 77.975) (xy 116.02 77.975) (xy 116.02 109.025) (xy 94.975 109.025)
 			)
 		)
