File: bq25798/bq25798.kicad_sch (KiCad schematic)
At the start: 0 parts

Commit message: Added schematics, needs adjustment for proper testing
Parts:
- added C29, C32: 47nF/10V, Capacitor_SMD:C_0201_0603Metric, symbol Device:C
- added C30, C36, C46, C54: 100nF/25V, Capacitor_SMD:C_0402_1005Metric, symbol Device:C
- added C31, C34, C38, C39, C41, C43, C45, C48, C49, C50, C51, C52: 10uF/25V, Capacitor_SMD:C_0805_2012Metric, symbol Device:C
- added C33: 4.7uF/10V, Capacitor_SMD:C_0402_1005Metric, symbol Device:C
- added C42: 1uF/16V, Capacitor_SMD:C_0603_1608Metric, symbol Device:C
- added CN2: B3P-VH, easyeda_import:CONN-TH_B3P-VH-LF-SN, symbol easyeda_import:B3P-VH
- added L3: 1uH, Inductor_SMD:L_1008_2520Metric, symbol Device:L
- added Q3: CH221K, easyeda_import:SOT-23-6_L2.9-W1.6-P0.95-LS2.8-BL-2, symbol easyeda_import:CH221K
- added Q4: HT04N200S, Package_TO_SOT_SMD:SOT-223, symbol Transistor_FET:2N7002
- added R14: 6.04kR/±1%, Resistor_SMD:R_0603_1608Metric, symbol Device:R
- added R15: 100R/±1%, Resistor_SMD:R_0805_2012Metric, symbol Device:R
- added R16: 1kR/±1%, Resistor_SMD:R_0603_1608Metric, symbol Device:R
- added R17: 8.25kR/±1%, Resistor_SMD:R_0603_1608Metric, symbol Device:R
- added R18: 17.4kR/±1%, Resistor_SMD:R_0603_1608Metric, symbol Device:R
- added R20: 5.23kR/±1%, Resistor_SMD:R_0402_1005Metric, symbol Device:R
- added R21: 30.9kR/±1%, Resistor_SMD:R_0603_1608Metric, symbol Device:R
- added R22: 20kR/±1%, Resistor_SMD:R_0603_1608Metric, symbol Device:R
- added R23, R24: 5.1kR/±1%, Resistor_SMD:R_0603_1608Metric, symbol Device:R
- added SW2: B3U-1000P, easyeda_import:KEY-SMD_B3U-1000PM, symbol easyeda_import:B3U-1000P
- added U4: R+O SMBJ6.0CA, Diode_SMD:D_SMB, symbol TVS diode:ESDBW5V0A1_C5173252
- added U5: BQ25798RQMR, easyeda_import:QFN-29_L4.0-W4.0-P0.40-TL-BQ25792RQMR, symbol easyeda_import:BQ25798RQMR
- added USBC2: MC-311D, easyeda_import:USB-C-SMD_MC-311D, symbol easyeda_import:MC-311D
Connections:
- new net: R14.1, U5.20 (PROG)
- new net: C42.1, Q3.1 (VDD), R16.2, R22.2
- new net: Q3.6 (CFG), R22.1
- new net: R15.1, U5.18 (BATP)
- new net +9V: C30.1, C31.1, C34.1, R16.1, U4.1 (K), U5.2 (VBUS), U5.3 (VBUS), U5.8 (VAC2), U5.9 (VAC1), USBC2.A4-B9 (VBUS), USBC2.B4-A9 (VBUS)
- new net BAT: C41.1, C45.1, Q4.2 (S), U5.22 (BAT), U5.23 (BAT)
- new net BTST1: C29.2, U5.4 (BTST1)
- new net BTST2: C32.2, U5.19 (BTST2)
- new net Battery+: CN2.3, Q4.3 (D), R15.2
- new net CC1: Q3.4 (CC1), R24.2, USBC2.A5 (CC1)
- new net CC2: Q3.5 (CC2), R23.2, USBC2.B5 (CC2)
- new net GND: C30.2, C31.2, C33.1, C34.2, C36.1, C38.1, C39.1, C41.2, C42.2, C43.1, C45.2, C46.2, C48.2, C49.2, C50.2, C51.2, C52.2, C54.2, CN2.1, Q3.2 (GND), R14.2, R18.2, R21.2, R23.1, R24.1, SW2.2, U4.2 (A), U5.10 (ACDRV2), U5.11 (ACDRV1), U5.13 (~{CE}), U5.27 (GND), USBC2.1 (SHIELD), USBC2.2 (SHIELD), USBC2.3 (SHIELD), USBC2.4 (SHIELD), USBC2.A1-B12 (GND), USBC2.B1-A12 (GND)
- new net ILIM_HIZ: R17.2, R18.1, U5.17 (ILIM_HIZ)
- new net INT: U5.21 (~{INT})
- new net NTC: CN2.2, R20.2, R21.1, U5.16 (TS)
- new net PMID: C36.2, C38.2, C39.2, C43.2, U5.29 (PMID)
- new net QON: C54.1, SW2.1, U5.12 (~{QON})
- new net REGN: C33.2, R17.1, R20.1, U5.5 (REGN)
- new net SCL1: U5.14 (SCL)
- new net SDA1: U5.15 (SDA)
- new net SDRV: Q4.1 (G), U5.24 (SDRV)
- new net SW1: C29.1, L3.1, U5.28 (SW1)
- new net SW2: C32.1, L3.2, U5.26 (SW2)
- new net SYS: C46.1, C48.1, C49.1, C50.1, C51.1, C52.1, U5.25 (SYS)
- no-connect marks 0 -> 9
Other:
- added sheet Input Buck (input_buck.kicad_sch)
- note added: "2.99A Input current limit"
- note added: "Battery should be 7.4V nominal"
- note added: "Most PD compliant devices at 5V can only negotiate up to 3A where as the Crowdspec device needs up to 5A (25W) to be stable. To get around this limitation, we can instead negotiate for 9V 3A (27W) to get the same energy density with less current. Since the Compute Module 5 cannot negotiate for 9V 3A, we have to implement the negotiation and override the expected handshake of the CM5."
- note added: "Override the CM5's EEPROM using PSU_MAX_CURRENT=5000"
- note added: "PD sink controller (9V)"
- note added: "QON pin(Internally pulled up) - Low for atleast 15ms = Exit shipping mode - Low for atleast 10s = IC hardware reset"
- note added: "The sink controller negotiates for 9V 3A where it then is recieved by the BQ25798. It automatically bucks the 9V down to the 7.4V voltage of the battery. This allows the IC to safely charge the battery. The BQ25798's SYS outupt voltage is dependent on the battery voltage. With the output current limit at 5A, it is better for us to buck down from a higher voltage rather than boosting from a lower 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"
- note added: "USB-C Power input interface"
